File: kicad/smarter-ac-unit.kicad_sch (KiCad schematic)
At the start: 8 parts

Commit message: fixes schematic and adds part list
Parts:
- R1: renamed from R?; value R_US -> 10K
- R2, R3: renamed from R?; value R_US -> 470
- gave numbers to parts that had none: 5
Changed lines of the file:
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@@
   (symbol (lib_id "power:+3.3V") (at 187.96 107.95 270) (unit 1)
     (in_bom yes) (on_board yes) (fields_autoplaced)
-    (property "Reference" "#PWR?" (id 0) (at 184.15 107.95 0)
+    (property "Reference" "#PWR05" (id 0) (at 184.15 107.95 0)
       (effects (font (size 1.27 1.27)) hide)
     )
@@
   (symbol (lib_id "Device:R_US") (at 179.07 93.98 180) (unit 1)
     (in_bom yes) (on_board yes) (fields_autoplaced)
-    (property "Reference" "R?" (id 0) (at 181.61 92.7099 0)
-      (effects (font (size 1.27 1.27)) (justify right))
-    )
-    (property "Value" "R_US" (id 1) (at 181.61 95.2499 0)
+    (property "Reference" "R3" (id 0) (at 181.61 92.7099 0)
+      (effects (font (size 1.27 1.27)) (justify right))
+    )
+    (property "Value" "470" (id 1) (at 181.61 95.2499 0)
       (effects (font (size 1.27 1.27)) (justify right))
     )
@@
   (symbol (lib_id "power:+3.3V") (at 187.96 43.18 270) (unit 1)
     (in_bom yes) (on_board yes) (fields_autoplaced)
-    (property "Reference" "#PWR?" (id 0) (at 184.15 43.18 0)
+    (property "Reference" "#PWR03" (id 0) (at 184.15 43.18 0)
       (effects (font (size 1.27 1.27)) hide)
     )
@@
   (symbol (lib_id "power:+3.3V") (at 102.87 93.98 0) (unit 1)
     (in_bom yes) (on_board yes) (fields_autoplaced)
-    (property "Reference" "#PWR?" (id 0) (at 102.87 97.79 0)
+    (property "Reference" "#PWR01" (id 0) (at 102.87 97.79 0)
       (effects (font (size 1.27 1.27)) hide)
     )
@@
   (symbol (lib_id "power:GND") (at 187.96 116.84 90) (unit 1)
     (in_bom yes) (on_board yes) (fields_autoplaced)
-    (property "Reference" "#PWR?" (id 0) (at 194.31 116.84 0)
+    (property "Reference" "#PWR06" (id 0) (at 194.31 116.84 0)
       (effects (font (size 1.27 1.27)) hide)
     )
@@
   (symbol (lib_id "Device:R_US") (at 170.18 64.77 0) (unit 1)
     (in_bom yes) (on_board yes) (fields_autoplaced)
-    (property "Reference" "R?" (id 0) (at 172.72 63.4999 0)
-      (effects (font (size 1.27 1.27)) (justify left))
-    )
-    (property "Value" "R_US" (id 1) (at 172.72 66.0399 0)
+    (property "Reference" "R2" (id 0) (at 172.72 63.4999 0)
+      (effects (font (size 1.27 1.27)) (justify left))
+    )
+    (property "Value" "470" (id 1) (at 172.72 66.0399 0)
       (effects (font (size 1.27 1.27)) (justify left))
     )
@@
   (symbol (lib_id "power:GND") (at 187.96 87.63 90) (unit 1)
     (in_bom yes) (on_board yes) (fields_autoplaced)
-    (property "Reference" "#PWR?" (id 0) (at 194.31 87.63 0)
+    (property "Reference" "#PWR04" (id 0) (at 194.31 87.63 0)
       (effects (font (size 1.27 1.27)) hide)
     )
@@
   (symbol (lib_id "Device:LED") (at 168.91 99.06 180) (unit 1)
     (in_bom yes) (on_board yes) (fields_autoplaced)
-    (property "Reference" "D?" (id 0) (at 170.4975 91.44 0))
+    (property "Reference" "D1" (id 0) (at 170.4975 91.44 0))
     (property "Value" "LED" (id 1) (at 170.4975 93.98 0))
     (property "Footprint" "" (id 2) (at 168.91 99.06 0)
@@
   (symbol (lib_id "Device:LED") (at 170.18 52.07 90) (unit 1)
     (in_bom yes) (on_board yes) (fields_autoplaced)
-    (property "Reference" "D?" (id 0) (at 177.8 53.6575 0))
+    (property "Reference" "D2" (id 0) (at 177.8 53.6575 0))
     (property "Value" "IR_LED" (id 1) (at 175.26 53.6575 0))
     (property "Footprint" "" (id 2) (at 170.18 52.07 0)
@@
   (symbol (lib_id "Switch:SW_Push") (at 144.78 53.34 0) (unit 1)
     (in_bom yes) (on_board yes) (fields_autoplaced)
-    (property "Reference" "SW?" (id 0) (at 144.78 45.72 0))
+    (property "Reference" "SW1" (id 0) (at 144.78 45.72 0))
     (property "Value" "SW_Push" (id 1) (at 144.78 48.26 0))
     (property "Footprint" "" (id 2) (at 144.78 48.26 0)
@@
   (symbol (lib_id "power:GND") (at 134.62 53.34 270) (unit 1)
     (in_bom yes) (on_board yes) (fields_autoplaced)
-    (property "Reference" "#PWR?" (id 0) (at 128.27 53.34 0)
+    (property "Reference" "#PWR02" (id 0) (at 128.27 53.34 0)
       (effects (font (size 1.27 1.27)) hide)
     )
@@
   (symbol (lib_id "Device:R_US") (at 162.56 43.18 90) (unit 1)
     (in_bom yes) (on_board yes) (fields_autoplaced)
-    (property "Reference" "R?" (id 0) (at 162.56 36.83 90))
-    (property "Value" "R_US" (id 1) (at 162.56 39.37 90))
+    (property "Reference" "R1" (id 0) (at 162.56 36.83 90))
+    (property "Value" "10K" (id 1) (at 162.56 39.37 90))
     (property "Footprint" "" (id 2) (at 162.814 42.164 90)
       (effects (font (size 1.27 1.27)) hide)
@@
   (symbol (lib_id "ESP8266:NodeMCU_1.0_(ESP-12E)") (at 130.81 90.17 0) (unit 1)
     (in_bom yes) (on_board yes) (fields_autoplaced)
-    (property "Reference" "U?" (id 0) (at 130.81 62.23 0)
+    (property "Reference" "U1" (id 0) (at 130.81 62.23 0)
       (effects (font (size 1.524 1.524)))
     )
@@
   (symbol (lib_id "Transistor_BJT:2N3904") (at 167.64 77.47 0) (unit 1)
     (in_bom yes) (on_board yes) (fields_autoplaced)
-    (property "Reference" "Q?" (id 0) (at 172.72 76.1999 0)
+    (property "Reference" "Q1" (id 0) (at 172.72 76.1999 0)
       (effects (font (size 1.27 1.27)) (justify left))
     )
@@
   )
   (symbol_instances
+    (path "/357f0f6b-0ae6-4fa5-8fda-06f38316ad2d"
+      (reference "#PWR01") (unit 1) (value "+3.3V") (footprint "")
+    )
+    (path "/d44b75c4-639b-4351-a377-f5c554c826be"
+      (reference "#PWR02") (unit 1) (value "GND") (footprint "")
+    )
+    (path "/318e0ae0-40d3-4c53-a77b-47c0f75cc6da"
+      (reference "#PWR03") (unit 1) (value "+3.3V") (footprint "")
+    )
+    (path "/643874cf-3107-4159-b5da-6872ef3fd9ce"
+      (reference "#PWR04") (unit 1) (value "GND") (footprint "")
+    )
     (path "/02d90c9c-ea2c-4c62-b6f2-a546f9c1c805"
-      (reference "#PWR?") (unit 1) (value "+3.3V") (footprint "")
-    )
-    (path "/318e0ae0-40d3-4c53-a77b-47c0f75cc6da"
-      (reference "#PWR?") (unit 1) (value "+3.3V") (footprint "")
-    )
-    (path "/357f0f6b-0ae6-4fa5-8fda-06f38316ad2d"
-      (reference "#PWR?") (unit 1) (value "+3.3V") (footprint "")
+      (reference "#PWR05") (unit 1) (value "+3.3V") (footprint "")
     )
     (path "/4eefc315-9c81-4d6c-af11-6b1452dcaa72"
-      (reference "#PWR?") (unit 1) (value "GND") (footprint "")
-    )
-    (path "/643874cf-3107-4159-b5da-6872ef3fd9ce"
-      (reference "#PWR?") (unit 1) (value "GND") (footprint "")
-    )
-    (path "/d44b75c4-639b-4351-a377-f5c554c826be"
-      (reference "#PWR?") (unit 1) (value "GND") (footprint "")
+      (reference "#PWR06") (unit 1) (value "GND") (footprint "")
     )
     (path "/7c1419d1-5adb-475a-8e57-89fe1d2fcc37"
-      (reference "D?") (unit 1) (value "LED") (footprint "")
+      (reference "D1") (unit 1) (value "LED") (footprint "")
     )
     (path "/88f2c724-5b23-4e5a-a011-c4f7ad4c066d"
-      (reference "D?") (unit 1) (value "IR_LED") (footprint "")
+      (reference "D2") (unit 1) (value "IR_LED") (footprint "")
     )
     (path "/f2e4c2e2-965f-47fa-b2ed-42debdfb6a8c"
-      (reference "Q?") (unit 1) (value "2N3904") (footprint "Package_TO_SOT_THT:TO-92_Inline")
+      (reference "Q1") (unit 1) (value "2N3904") (footprint "Package_TO_SOT_THT:TO-92_Inline")
+    )
+    (path "/df0f5a9c-974e-4cc5-8cb9-8a5f80f11d80"
+      (reference "R1") (unit 1) (value "10K") (footprint "")
+    )
+    (path "/5efd316f-bac9-4d4b-b474-ab6afd0f34ed"
+      (reference "R2") (unit 1) (value "470") (footprint "")
     )
     (path "/15a41ed9-4820-472d-a12a-683e3cb1054a"
-      (reference "R?") (unit 1) (value "R_US") (footprint "")
-    )
-    (path "/5efd316f-bac9-4d4b-b474-ab6afd0f34ed"
-      (reference "R?") (unit 1) (value "R_US") (footprint "")
-    )
-    (path "/df0f5a9c-974e-4cc5-8cb9-8a5f80f11d80"
-      (reference "R?") (unit 1) (value "R_US") (footprint "")
+      (reference "R3") (unit 1) (value "470") (footprint "")
     )
     (path "/8f63fef0-06a0-4360-bde5-89c5d3255508"
-      (reference "SW?") (unit 1) (value "SW_Push") (footprint "")
+      (reference "SW1") (unit 1) (value "SW_Push") (footprint "")
     )
     (path "/eb01c17c-3d7f-4466-a855-1a70b3706ba9"
-      (reference "U?") (unit 1) (value "NodeMCU_1.0_(ESP-12E)") (footprint "")
-    )
-  )
+      (reference "U1") (unit 1) (value "NodeMCU_1.0_(ESP-12E)") (footprint "")
+    )
+  )

Commit message: re-export all cad
Parts:
- R2: value 470 -> 47
Changed lines of the file:
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@@
       (effects (font (size 1.27 1.27)) (justify left))
     )
-    (property "Value" "470" (id 1) (at 172.72 66.0399 0)
+    (property "Value" "47" (id 1) (at 172.72 66.0399 0)
       (effects (font (size 1.27 1.27)) (justify left))
     )
@@
     )
     (path "/5efd316f-bac9-4d4b-b474-ab6afd0f34ed"
-      (reference "R2") (unit 1) (value "470") (footprint "")
+      (reference "R2") (unit 1) (value "47") (footprint "")
     )
     (path "/15a41ed9-4820-472d-a12a-683e3cb1054a"
